File: pcb/vestee main.brd (EAGLE design)
At the start: 65 x 65 mm, 39 parts, among them IC1 LD117AS12TR, IC2 FT232RL, Q1 MMBT2222A, Q3 MMBT4403

Commit message: pcb rev3
Parts:
- removed C6: 100nF, SparkFun-Capacitors:0805-CAP
- removed DBG_TX, DBG_TX1, PAD1, PAD2, PAD5: (no value), wirepad:SMD1,27-2,54
- removed IC2: FT232RL, ftdichip:SSOP28
- removed LED4: (no value), led:SML0805
- removed R16, R18, R19: (no value), rcl:R0805
- added C1: (no value), SparkFun-Passives:EIA3528
- added C7, C8: 100nF, rcl:C0603
- added D1, D2, D4, D5, D6, D7, D8: KPBA-3010ESGC, SparkFun-LED:APA3010SF4C
- added IC3: CP210X_USB_UART, SparkFun-DigitalIC:MLP28
- added PRPIHERALS1: AUDIO-JACK-2.5-CUI, SparkFun-Connectors:STEREOJACK2.5_SMD_CUI
- added R30, R31: 12k, rcl:R0603
- added U$3, U$4: SCT2024CSSG, vestee:SSOP24
- C2: value (none) -> 100nF; device SparkFun-Capacitors:PANASONIC_D -> rcl:C0603
- C3: device SparkFun-Capacitors:0805-CAP -> rcl:C0603
- C4: value 10nF -> 10n; device SparkFun-Capacitors:0805-CAP -> rcl:C0603
- C5: value 100nF -> 100n; device SparkFun-Capacitors:0805-CAP -> rcl:C0603
- D3: value (none) -> KPBA-3010ESGC; device diode:SOD80C -> SparkFun-LED:APA3010SF4C
- Q3: value MMBT4403 -> MMBT2222A
- R1, R12, R2, R20, R21, R3, R7: device rcl:R0805 -> rcl:R0603
- R10, R11, R6, R9: value (none) -> 12k; device rcl:R0805 -> rcl:R0603
- R14, R8: value (none) -> 470R; device rcl:R0805 -> rcl:R0603
- R15: value (none) -> 470; device rcl:R0805 -> rcl:R0603
- U$2: value (none) -> KCDA02-103; device DHT11:DHT11 -> vestee:KCDA02-103
- moved U$2 43.6 mm to (32.5, 52.0), turned to 0 degrees
- moved Q3 34.4 mm to (28.0, 41.4), turned to 270 degrees
- moved R14 32.8 mm to (29.0, 26.5)
- moved C2 31.1 mm to (37.0, 38.5), turned to 270 degrees
- moved R6 30.1 mm to (22.0, 26.5), turned to 90 degrees
- moved R2 28.4 mm to (39.0, 26.5), turned to 270 degrees
- moved R3 25.9 mm to (24.0, 38.5)
- moved R15 24.6 mm to (54.0, 43.0), turned to 0 degrees
- moved R12 22.6 mm to (24.0, 26.5), turned to 90 degrees
- moved Q1 21.8 mm to (28.0, 38.3), turned to 270 degrees
- moved R1 20.7 mm to (22.0, 38.5), turned to 90 degrees
- moved R11 18.9 mm to (39.0, 38.5)
- moved C5 18.9 mm to (16.0, 31.5)
- moved R9 17.4 mm to (31.0, 26.5)
- moved R10 16.0 mm to (35.0, 38.5), turned to 270 degrees
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Connections:
- net N$19 renamed SWITCH
- removed net ELECTRODE: R15.1, U$1.GPIO4
- removed net FLED: R6.2, U$1.GPIO12
- removed net N$1: R1.1, R18.1, U$1.GPIO14
- removed net N$10: Q1.1, R14.1, R6.1
- removed net N$16: LED4.C, Q1.3
- removed net N$17: PAD2.1, Q3.3
- removed net N$21: R10.1, U$1.CH_PD
- removed net N$26: PAD1.1, R19.1
- removed net N$27: Q3.1, R15.2, R16.1
- removed net N$4: R12.2, R2.1, U$1.GPIO16
- removed net N$6: R18.2, U$2.DATA
- new net A1: U$2.17, U$3.7
- new net A2: U$2.12, U$3.11
- new net B1: U$2.16, U$3.8
- new net B2: U$2.11, U$3.12
- new net C1: U$2.4, U$3.18
- new net C2: U$2.9, U$3.14
- new net CH_PD: R11.1, U$1.CH_PD
- new net CLK: U$1.GPIO13, U$3.3
- new net D1: U$2.2, U$3.19
- new net D1G: D1.3, U$4.12
- new net D1R: D1.2, U$4.11
- new net D2: U$2.7, U$3.15
- new net D2G: D2.3, U$4.10
- new net D2R: D2.2, U$4.9
- new net D3G: D3.3, U$4.8
- new net D3R: D3.2, U$4.7
- new net D4G: D4.3, U$4.6
- new net D4R: D4.2, U$4.5
- new net D5G: D5.3, U$4.19
- new net D5R: D5.2, U$4.20
- new net D6G: D6.3, U$4.18
- new net D6R: D6.2, U$4.17
- new net D7G: D7.3, U$4.16
- new net D7R: D7.2, U$4.15
- new net D8G: D8.3, U$4.14
- new net D8R: D8.2, U$4.13
- new net DP1: U$2.5, U$3.17
- new net DP2: U$2.10, U$3.13
- new net E1: U$2.1, U$3.20
- new net E2: U$2.6, U$3.16
- new net F1: U$2.19, U$3.6
- new net F2: U$2.14, U$3.10
- new net G1: U$2.20, U$3.5
- new net G2: U$2.15, U$3.9
- new net GPIO0: Q1.3, R30.1, R7.2, U$1.GPIO0
- new net GPIO16: R15.1, U$1.GPIO16
- new net GPIO2: R31.1, U$1.GPIO2
- new net JACK: PRPIHERALS.3, PRPIHERALS1.3, R12.1
- new net LA/: U$1.GPIO4, U$3.4
- new net N$14: IC3.9, R6.2
- new net REST: C2.1, Q3.3, R10.1, R15.2, U$1.REST
- new net SDI: U$1.GPIO12, U$4.2
- new net SDO: U$3.2, U$4.22
- new net TXD: IC3.26, R14.2
- net 1-WIRE: now also R12.2, R2.1, U$1.GPIO15; no longer PRPIHERALS.3, R12.1
- net ADC: no longer D3.C, R19.2
- net DTR: now also IC3.28, Q1.2, R1.1; no longer IC2.2, R3.2, U$1.GPIO0
- net FTDI_RXD: now also IC3.25; no longer IC2.5
- net FTDI_TXD: now also R14.1; no longer IC2.1
- net GND: now also C1.C, C2.2, C7.2, C8.2, IC3.3, IC3.EXP, IC3.M, PRPIHERALS1.1, U$3.1, U$4.1; no longer C2.-, C6.1, D3.A, DBG_TX1.1, IC2.18, IC2.21, IC2.25, IC2.26, IC2.7, PAD5.1, Q1.2, R14.2, U$1.GPIO15, U$2.GND
- net N$15: now also Q1.1, R3.2; no longer LED4.A, R7.1
- net N$28: now also IC3.4; no longer IC2.15
- net N$29: now also IC3.5; no longer IC2.16
- net N$5: now also Q3.1, R1.2; no longer DBG_TX.1, U$1.GPIO2
- net N$9: now also IC3.6; no longer IC2.17
- net RTS: now also IC3.24, Q3.2, R3.1; no longer IC2.3, R11.1, U$1.REST
- net VCC: now also C1.A, C7.1, C8.1, D1.COM, D2.COM, D3.COM, D4.COM, D5.COM, D6.COM, D7.COM, D8.COM, PRPIHERALS1.2, R30.2, R31.2, R6.1, R7.1, U$2.13, U$2.18, U$2.3, U$2.8, U$3.24, U$4.24; no longer C2.+, C6.2, IC2.4, Q3.2, R1.2, R16.2, R3.1, R7.2, U$2.VCC
- net VIN: now also IC3.7, IC3.8; no longer IC2.20
Routing:
- net VCC: track 182.1 -> 383.6 mm, vias 4 -> 19
- net D1G: track 0.00 -> 73.6 mm, vias 0 -> 2
- net D1R: track 0.00 -> 71.1 mm, vias 0 -> 2
- net N$6: track 70.4 -> 0.00 mm, vias 2 -> 0
- net D2G: track 0.00 -> 58.3 mm, vias 0 -> 2
- net D2R: track 0.00 -> 56.0 mm, vias 0 -> 2
- net JACK: track 0.00 -> 47.2 mm, vias 0 -> 2
- net N$26: track 46.1 -> 0.00 mm, vias 2 -> 0
- net D3G: track 0.00 -> 45.3 mm, vias 0 -> 2
- net D3R: track 0.00 -> 44.4 mm, vias 0 -> 2
- net N$4: track 44.2 -> 0.00 mm, vias 2 -> 0
- net D4R: track 0.00 -> 43.5 mm, vias 0 -> 3
- net SDO: track 0.00 -> 42.8 mm, vias 0 -> 2
- net GPIO0: track 0.00 -> 42.7 mm, vias 0 -> 2
- net D4G: track 0.00 -> 39.6 mm, vias 0 -> 2
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Other:
- board size 65 x 65 mm -> 57.4 x 63.6 mm
- board text removed: "and"
- board text removed: "vestee.io"

Commit message: Added current setting resistors for LED drivers
Parts:
- added R4, R5: (no value), rcl:R0603
- moved C8 1.15 mm to (51.6, 12.4)
- moved C7 0.51 mm to (51.5, 49.0)
Connections:
- new net N$1: R4.1, U$3.23
- new net N$4: R5.1, U$4.23
- net GND: now also R4.2, R5.2
Routing:
- net N$4: track 0.00 -> 7.25 mm
- net N$1: track 0.00 -> 5.72 mm
- net VCC: track 383.6 -> 384.9 mm, vias 19 -> 20
- net GND: vias 30 -> 31
Changed lines of the file:
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@@
 <setting verticaltext="up"/>
 </settings>
-<grid distance="10" unitdist="mil" unit="mm" style="lines" multiple="1" display="yes" altdistance="0.01" altunitdist="mm" altunit="mm"/>
+<grid distance="10" unitdist="mil" unit="mil" style="lines" multiple="1" display="yes" altdistance="0.01" altunitdist="mm" altunit="mm"/>
 <layers>
 <layer number="1" name="Top" color="4" fill="1" visible="yes" active="yes"/>
@@
 <element name="C2" library="rcl" package="C0603" value="100nF" x="37" y="38.5" rot="R270"/>
 <element name="U$4" library="vestee" package="SSOP24" value="SCT2024CSSG" x="46" y="15" rot="R180"/>
-<element name="C7" library="rcl" package="C0603" value="100nF" x="51.5" y="48.5" rot="R90"/>
-<element name="C8" library="rcl" package="C0603" value="100nF" x="51.5" y="13.5" rot="R90"/>
+<element name="C7" library="rcl" package="C0603" value="100nF" x="51.5" y="49.008" rot="R90"/>
+<element name="C8" library="rcl" package="C0603" value="100nF" x="51.6" y="12.352" rot="R90"/>
+<element name="R4" library="rcl" package="R0603" value="" x="54.002" y="46.632"/>
+<element name="R5" library="rcl" package="R0603" value="" x="54.21" y="12.356" rot="R90"/>
 </elements>
 <signals>
@@
 <via x="53.848" y="49.784" extent="1-16" drill="0.3048" shape="octagon"/>
 <via x="53.848" y="48.768" extent="1-16" drill="0.3048" shape="octagon"/>
+<contactref element="R4" pad="2"/>
+<contactref element="R5" pad="2"/>
+<via x="56.388" y="46.736" extent="1-16" drill="0.3048" shape="octagon"/>
 </signal>
 <signal name="VCC">
@@
 <contactref element="C8" pad="1"/>
 <contactref element="U$4" pad="24"/>
-<wire x1="49.4925" y1="47" x2="50.1425" y2="47.65" width="0.2032" layer="1"/>
-<wire x1="50.1425" y1="47.65" x2="51.5" y2="47.65" width="0.2032" layer="1"/>
-<wire x1="51.5" y1="47.65" x2="51.652" y2="47.498" width="0.2032" layer="1"/>
-<wire x1="51.652" y1="47.498" x2="58.928" y2="47.498" width="0.2032" layer="1"/>
-<wire x1="58.928" y1="47.498" x2="60.452" y2="45.974" width="0.2032" layer="1"/>
+<wire x1="49.4925" y1="47" x2="50.6505" y2="48.158" width="0.2032" layer="1"/>
+<wire x1="58.42" y1="48.006" x2="60.452" y2="45.974" width="0.2032" layer="1"/>
 <wire x1="60.452" y1="45.974" x2="60.452" y2="43.942" width="0.2032" layer="1"/>
-<wire x1="49.4925" y1="12" x2="50.1425" y2="12.65" width="0.2032" layer="1"/>
-<wire x1="50.1425" y1="12.65" x2="51.5" y2="12.65" width="0.2032" layer="1"/>
-<wire x1="51.5" y1="12.65" x2="52.02" y2="12.65" width="0.2032" layer="1"/>
-<wire x1="52.02" y1="12.65" x2="58.42" y2="19.05" width="0.2032" layer="1"/>
 <wire x1="58.42" y1="19.05" x2="58.467009375" y2="19.05" width="0.2032" layer="1"/>
 <wire x1="58.467009375" y1="19.05" x2="58.8344375" y2="19.417428125" width="0.2032" layer="1"/>
@@
 <wire x1="36.328" y1="45.302" x2="36.322" y2="45.296" width="0.2032" layer="16"/>
 <wire x1="36.322" y1="45.296" x2="36.322" y2="45.212" width="0.2032" layer="16"/>
+<wire x1="50.6505" y1="48.158" x2="51.5" y2="48.158" width="0.2032" layer="1"/>
+<wire x1="58.42" y1="48.006" x2="51.652" y2="48.006" width="0.2032" layer="1"/>
+<wire x1="51.652" y1="48.006" x2="51.5" y2="48.158" width="0.2032" layer="1"/>
+<wire x1="49.4925" y1="11.9755" x2="49.4925" y2="12" width="0.2032" layer="1"/>
+<wire x1="51.528" y1="11.43" x2="51.6" y2="11.502" width="0.2032" layer="1"/>
+<via x="52.716" y="11.016" extent="1-16" drill="0.3048" shape="octagon"/>
+<wire x1="52.716" y1="11.016" x2="52.23" y2="11.502" width="0.254" layer="1"/>
+<wire x1="52.23" y1="11.502" x2="51.6" y2="11.502" width="0.254" layer="1"/>
+<wire x1="51.528" y1="11.43" x2="50.958" y2="12" width="0.254" layer="1"/>
+<wire x1="50.958" y1="12" x2="49.4925" y2="12" width="0.254" layer="1"/>
+<wire x1="45.212" y1="6.096" x2="52.716" y2="11.016" width="0.2032" layer="16" curve="13.506076"/>
 </signal>
 <signal name="1-WIRE">
@@
 <wire x1="31.78" y1="45.6392" x2="31.78" y2="47.04" width="0.2032" layer="1"/>
 </signal>
+<signal name="N$1">
+<contactref element="U$3" pad="23"/>
+<contactref element="R4" pad="1"/>
+<wire x1="48.8575" y1="47" x2="48.8575" y2="45.9625" width="0.2032" layer="1"/>
+<wire x1="48.8575" y1="45.9625" x2="48.99" y2="45.83" width="0.2032" layer="1"/>
+<wire x1="48.99" y1="45.83" x2="52.35" y2="45.83" width="0.2032" layer="1"/>
+<wire x1="52.35" y1="45.83" x2="53.152" y2="46.632" width="0.2032" layer="1"/>
+</signal>
+<signal name="N$4">
+<contactref element="U$4" pad="23"/>
+<contactref element="R5" pad="1"/>
+<wire x1="48.8575" y1="12" x2="48.8575" y2="11.1325" width="0.2032" layer="1"/>
+<wire x1="48.8575" y1="11.1325" x2="49.576" y2="10.414" width="0.2032" layer="1"/>
+<wire x1="49.576" y1="10.414" x2="53.594" y2="10.414" width="0.2032" layer="1"/>
+<wire x1="53.594" y1="10.414" x2="54.21" y2="11.03" width="0.2032" layer="1"/>
+<wire x1="54.21" y1="11.03" x2="54.21" y2="11.506" width="0.2032" layer="1"/>
+</signal>
 </signals>
